Commit message: feat: add suction grasp pick and place flow

File: src/python/arcor2_ur/data/urdf/ur5e.urdf (robot description, URDF)
Before this commit: robot ur5e, 13 links, 12 joints
Links:
- added link suction_base_link; visual mesh filename=package://meshes/ur5e/collision/base_link_1cup.stl
- added link suction_cup_link; visual mesh filename=package://meshes/ur5e/collision/suction_cup_1cup.stl
- added link suction_tcp
Joints:
- added joint suction_base_to_cup: type fixed, parent suction_base_link, child suction_cup_link, origin xyz=0 0 0.188 rpy=0 0 0
- added joint suction_cup_to_tcp: type fixed, parent suction_cup_link, child suction_tcp, origin xyz=0 0 0 rpy=0 0 0
- added joint tool0_to_suction_base: type fixed, parent tool0, child suction_base_link, origin xyz=0 0 0 rpy=0 0 0

Commit message: feat: optimize ros worker grasping
Add new grasp planner, update ROS worker grasp flow, and add pick-up tests.

File: src/python/arcor2_ur/data/urdf/ur5e.urdf (robot description, URDF)
Before this commit: robot ur5e, 16 links, 15 joints
Joints:
- joint suction_base_to_cup: origin xyz=0 0 0.188 rpy=0 0 0 -> xyz=0 0 0.19 rpy=0 0 0

Commit message: fix(arcor2_ur): improve UR5e suction and collision tests

File: src/python/arcor2_ur/data/urdf/ur5e.urdf (robot description, URDF)
Before this commit: robot ur5e, 16 links, 15 joints
Links:
- link suction_base_link: geometry collision mesh filename=package://meshes/ur5e/collision/base_link_1cup.stl; visual mesh filename=package://meshes/ur5e/collision/base_link_1cup.stl
- link suction_cup_link: geometry collision mesh filename=package://meshes/ur5e/collision/suction_cup_1cup.stl; visual mesh filename=package://meshes/ur5e/collision/suction_cup_1cup.stl
Joints:
- joint suction_base_to_cup: origin xyz=0 0 0.19 rpy=0 0 0 -> xyz=0 0 0.1025 rpy=0 0 0
